File: kicad/Signalgenerator/Signalgenerator.kicad_pcb (KiCad board)
At the start: 2 copper layers, 62 parts, among them J1 Conn_01x01, J2 Conn_01x01, SW1 OS103011MS8QP1, SW2 SW_DPDT_x2, SW3 OS103011MS8QP1, U1 LT1354CS8, U2 LT1354CS8, U3 LT1354CS8, U4 LT1354CS8, U5 LT1354CS8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

Commit message: stand jetzt
Parts:
- removed R14, R16, R18: 0, Resistor_SMD:R_0805_2012Metric_Pad1.20x1.40mm_HandSolder
- C12, C14: footprint Capacitor_SMD:C_0603_1608Metric_Pad1.08x0.95mm_HandSolder -> Capacitor_SMD:C_0805_2012Metric
- moved R15 21.1 mm to (29.0, 49.0)
- moved R17 20.5 mm to (44.0, 59.5)
- moved Dreieck1 15.3 mm to (57.0, 28.5)
- moved PWM1 14.1 mm to (68.0, 55.5)
- moved C8 12.1 mm to (69.0, 47.5)
- moved Rechteck1 11.7 mm to (34.0, 26.5)
- moved C23 10.7 mm to (53.5, 46.0), turned to 90 degrees
- moved C18 9.11 mm to (45.0, 35.0), turned to 90 degrees
- moved C12 8.94 mm to (53.5, 36.0), turned to 90 degrees
- moved C22 8.31 mm to (51.5, 46.0), turned to 90 degrees
- moved R2 8.18 mm to (35.0, 34.0)
- moved R1 8.16 mm to (43.0, 35.0)
- moved J2 7.23 mm to (22.0, 29.5)
- moved 10k1 7.08 mm to (75.1, 35.3)
- moved R11 7.08 mm to (69.6, 42.9)
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Connections:
- 22k1 pad 2: Net-(22k1-Pad2) -> Net-(U2--IN)
- C22 pad 1: Net-(22k1-Pad2) -> Net-(U2--IN)
- C23 pad 1: Net-(22k1-Pad2) -> Net-(U2--IN)
- C24 pad 2: Net-(22k1-Pad2) -> Net-(U2--IN)
- Dreieck1 pad 1: Net-(U5-+IN) -> Net-(U2-OUT)
- SW1 pad 2: Net-(U5-+IN) -> Net-(U2-OUT)
- SW3 pad 3: Net-(U5-+IN) -> Net-(U2-OUT)
- U3 pad 3: Net-(U3-+IN) -> Net-(U2-OUT)
- U5 pad 3: Net-(U5-+IN) -> Net-(U2-OUT)
Routing:
- net Ub-: track 52.1 -> 17.4 mm
- net GND: track 36.6 -> 7.19 mm
- net Net-(U2-OUT): track 9.12 -> 31.0 mm
- net Net-(U2--IN): track 4.86 -> 23.4 mm
- net Net-(U5-+IN): track 16.1 -> 0.00 mm
- net Net-(SW2A-B): track 16.9 -> 2.45 mm
- net Net-(22k1-Pad2): track 11.2 -> 0.00 mm
- net Net-(U1-OUT): track 10.3 -> 2.63 mm
- net Net-(U1-+IN): track 7.12 -> 0.00 mm
- net Net-(U3-+IN): track 5.50 -> 0.00 mm
- net Net-(22k1-Pad3): track 3.49 -> 0.00 mm
- net Ub+: track 39.7 -> 38.6 mm
- net Net-(C22-Pad2): track 3.05 -> 3.64 mm
- net Net-(C24-Pad1): track 4.18 -> 3.64 mm
