File: kicad/Signalgenerator/Signalgenerator.kicad_pcb (KiCad board)
At the start: 2 copper layers, 59 parts, among them J1 Conn_01x01, J2 Conn_01x01, SW1 OS103011MS8QP1, SW2 SW_DPDT_x2, SW3 OS103011MS8QP1, U1 LT1354CS8, U2 LT1354CS8, U3 LT1354CS8, U4 LT1354CS8, U5 LT1354CS8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

Commit message: changed changes
Parts:
- moved SW2 7.36 mm to (47.5, 27.5), turned to 0 degrees
- moved Rechteck1 7.16 mm to (31.0, 20.0)
- moved 22k2 3.54 mm to (40.0, 27.5)
- moved D1 3.41 mm to (47.5, 23.5), turned to 180 degrees
- moved R3 2.48 mm to (39.0, 30.0), turned to 180 degrees
- moved C18 1.00 mm to (45.0, 36.0)
- moved R1 1.00 mm to (43.0, 36.0)
- moved R2 1.00 mm to (35.0, 35.0)
- moved U1 1.00 mm to (39.2, 35.2)
- moved R4 0.50 mm to (39.0, 40.0)
Routing:
- net Ub+: track 38.6 -> 92.6 mm
- net Net-(SW2A-B): track 2.45 -> 16.1 mm
- net Net-(U1-+IN): track 0.00 -> 10.1 mm
- net Ub-: track 17.4 -> 25.2 mm
- net Net-(D1-A): track 9.41 -> 2.52 mm
- net Net-(U1-OUT): track 2.63 -> 9.33 mm
- net Net-(U2-OUT): track 31.0 -> 26.9 mm
- net Net-(22k1-Pad3): track 0.00 -> 3.19 mm
- net Net-(D1-K): track 4.81 -> 7.54 mm
- net Net-(U2--IN): track 23.4 -> 25.6 mm
- net Net-(SW2A-A): track 7.43 -> 6.88 mm

Commit message: did things
Parts:
- moved RV2 71.3 mm to (103.0, 33.0), turned to 180 degrees
- moved RV1 62.9 mm to (93.0, 33.0), turned to 180 degrees
- moved TP1 62.1 mm to (84.5, 21.5)
- moved R12 60.5 mm to (98.0, 37.5), turned to -90 degrees
- moved SW3 59.5 mm to (78.0, 43.5), turned to 90 degrees
- moved C16 54.6 mm to (78.0, 34.4), turned to 90 degrees
- moved U7 52.5 mm to (82.7, 36.9)
- moved R13 47.2 mm to (84.5, 47.0)
- moved C6 44.7 mm to (84.9, 49.0)
- moved R7 39.8 mm to (79.5, 50.5)
- moved U4 39.6 mm to (84.2, 52.9)
- moved C20 38.1 mm to (89.0, 53.9), turned to 90 degrees
- moved R17 29.4 mm to (66.5, 40.5), turned to 180 degrees
- moved U5 29.4 mm to (75.4, 52.3), turned to -90 degrees
- moved C10 20.9 mm to (74.1, 57.0), turned to 0 degrees
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Routing:
- net Ub+: track 92.6 -> 162.6 mm
- net Net-(U2-OUT): track 26.9 -> 65.2 mm
- net Ub-: track 25.2 -> 51.1 mm
- net Net-(U7--IN): track 0.00 -> 19.3 mm
- net Net-(U4-OUT): track 0.00 -> 11.6 mm
- net Net-(U6-+IN): track 0.00 -> 10.8 mm
- net Net-(U5--IN): track 0.00 -> 10.7 mm
- net Net-(U7-+IN): track 0.00 -> 7.40 mm
- net Net-(U7-OUT): track 0.00 -> 6.40 mm
- net Net-(U6-OUT): track 0.00 -> 4.96 mm
- net Net-(U6--IN): track 0.00 -> 4.86 mm
- net Net-(R12-Pad1): track 0.00 -> 3.13 mm
- net Net-(10k1-Pad3): track 0.00 -> 2.83 mm
- net Net-(10k1-Pad1): track 0.00 -> 2.68 mm
- net Net-(U4--IN): track 0.00 -> 2.30 mm
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
Commit message: done da ting
Parts:
- removed R17: 0, Resistor_SMD:R_0805_2012Metric_Pad1.20x1.40mm_HandSolder
- added R14: 0, Resistor_SMD:R_0805_2012Metric_Pad1.20x1.40mm_HandSolder, F.Cu at (80.5, 55.0)
- C12, C14: footprint Capacitor_SMD:C_0805_2012Metric -> Capacitor_SMD:C_0603_1608Metric_Pad1.08x0.95mm_HandSolder
- moved R15 40.5 mm to (69.5, 47.5), turned to 90 degrees
- moved PWM1 22.1 mm to (77.5, 40.0)
- moved RV2 21.5 mm to (94.0, 52.5)
- moved R12 8.73 mm to (90.0, 41.0), turned to 90 degrees
- moved RV1 2.00 mm to (95.0, 33.0)
- moved U4 1.43 mm to (85.4, 53.7), turned to 90 degrees
- moved C10 0.50 mm to (74.6, 57.0)
Routing:
- net Ub-: track 51.1 -> 192.7 mm
- net Ub+: track 162.6 -> 222.8 mm
- net Net-(U4--IN): track 2.30 -> 17.9 mm
- net Net-(U4-OUT): track 11.6 -> 7.91 mm
- net Net-(R12-Pad1): track 3.13 -> 0.00 mm
- net Net-(U2-OUT): track 65.2 -> 62.7 mm
- net Net-(U7-OUT): track 6.40 -> 8.40 mm
- net Net-(U7--IN): track 19.3 -> 17.8 mm

Commit message: U du da rest
Parts:
- moved RV2 3.00 mm to (94.0, 49.5)
Routing:
- net GND: track 7.19 -> 118.2 mm
- net Ub+: track 222.8 -> 240.9 mm
- net Net-(R12-Pad1): track 0.00 -> 10.6 mm
- net Ub-: track 192.7 -> 200.8 mm
